Commit message: astar tillagt

File: src/testrig/urdf/rig.urdf.xacro (robot description, xacro)
@@ -2,6 +2,7 @@
 <robot name="testrig" xmlns:xacro="http://ros.org/wiki/xacro">
   <xacro:include filename="$(find testrig)/urdf/common_properties.xacro"/>
-  <!-- <xacro:include filename="$(find hktest)/urdf/rig.gazebo.xacro"/>
-  <xacro:include filename="$(find hktest)/urdf/rig.transmission.xacro"/> -->
+  <xacro:include filename="$(find testrig)/urdf/rig.gazebo.xacro"/>
+  <xacro:include filename="$(find testrig)/urdf/rig.transmission.xacro"/>
+  <xacro:include filename="$(find velodyne_description)/urdf/VLP-16.urdf.xacro"/>
   <xacro:property name="z" value="0.360"/>
   <!-- LIDAR -->
@@ -42,4 +43,7 @@
   </link>
   <!-- LIDAR, CAMERA, IMU -->
+  <VLP-16 parent="base_link1" name="velodyne">
+    <origin xyz="0 0.13 0.75" rpy="0 0 0" />
+  </VLP-16>
   <joint name="camera_joint" type="fixed">
     <axis xyz="0 1 0" />
@@ -132,5 +136,5 @@
     <parent link="base_link1"/>
     <child link="front_link_middle"/>
-    <limit effort="1000" lower="-0.7" upper="0.7" velocity="0.5" />
+    <limit effort="1000" lower="-0.75" upper="0.75" velocity="0.5" />
     <origin xyz="0.0 -0.070 ${z-0.035}" rpy="1.57 0 0"/>
     <axis xyz="0 1 0"/>
@@ -249,5 +253,5 @@
     <parent link="middle_base" />
     <child link = "middle_link_back" />
-    <limit effort="1000" lower="-0.7" upper="0.7" velocity="0.5" />
+    <limit effort="1000" lower="-0.75" upper="0.75" velocity="0.5" />
     <origin xyz="0 -0.520 0" rpy="0 0 1.57" />
     <axis xyz="0 1 0"/>
@@ -361,7 +365,7 @@
       </inertial>
   </link>
-  <!-- <gazebo>
+  <gazebo>
 	<plugin name="gazebo_ros_control" filename="libgazebo_ros_control.so">
     </plugin>
-  </gazebo> -->
+  </gazebo>
 </robot>

Commit message: Project end upload

File: src/testrig/urdf/rig.urdf.xacro (robot description, xacro)
@@ -17,5 +17,5 @@
     <parent link="base_footprint"/>
     <child link="base_link1"/>
-    <origin xyz="0 0 0" rpy="0 0 0"/>
+    <origin xyz="0 -0.44 0" rpy="0 0 0"/>
   </joint>
 <!-- Front -->
